Commit message: fine tune the arm mass to make whole body get a neural bouyancy

File: hdt_description/urdf/hdt_angler_a_arm.xacro (robot description, xacro)
@@ -13,4 +13,5 @@
         <!-- constants -->
         <xacro:property name="M_PI" value="3.1415926535897931"/>
+        <xacro:property name="mass" value="0.107" />
         <xacro:property name="drive_length" value="0.047"/>
         <xacro:property name="a35_length" value="0.03855"/>
@@ -66,5 +67,5 @@
             <inertial>
                 <origin xyz="0 0 0" rpy="0 0 0"/>
-                <mass value="0.1"/>
+                <mass value="${mass}"/>
                 <xacro:default_inertia />
             </inertial>
@@ -95,5 +96,5 @@
             <inertial>
                 <origin xyz="0 0 0" rpy="0 0 0"/>
-                <mass value="0.1"/>
+                <mass value="${mass}"/>
                 <xacro:default_inertia />
             </inertial>
@@ -124,5 +125,5 @@
             <inertial>
                 <origin xyz="0 0 0" rpy="${M_PI} 0 0"/>
-                <mass value="0.1"/>
+                <mass value="${mass}"/>
                 <xacro:default_inertia />
             </inertial>
@@ -150,5 +151,5 @@
             <inertial>
                 <origin xyz="0 0 0" rpy="0 0 0"/>
-                <mass value="0.1"/>
+                <mass value="${mass}"/>
                 <xacro:default_inertia />
             </inertial>
@@ -176,5 +177,5 @@
             <inertial>
                 <origin xyz="0 0 0" rpy="0 ${M_PI} 0"/>
-                <mass value="0.1"/>
+                <mass value="${mass}"/>
                 <xacro:default_inertia />
             </inertial>
@@ -206,5 +207,5 @@
             <inertial>
                 <origin xyz="0 0 0" rpy="0 ${M_PI/2} -${M_PI/2}"/>
-                <mass value="0.1"/>
+                <mass value="${mass}"/>
                 <xacro:default_inertia />
             </inertial>
@@ -235,5 +236,5 @@
             <inertial>
                 <origin xyz="0 0 0" rpy="${M_PI} 0 0"/>
-                <mass value="0.1"/>
+                <mass value="${mass}"/>
                 <xacro:default_inertia />
             </inertial>
@@ -261,5 +262,5 @@
             <inertial>
                 <origin xyz="0 0 0" rpy="0 0 ${M_PI}"/>
-                <mass value="0.1"/>
+                <mass value="${mass}"/>
                 <xacro:default_inertia />
             </inertial>
@@ -290,5 +291,5 @@
             <inertial>
                 <origin xyz="0 0 0" rpy="0 0 0"/>
-                <mass value="0.1"/>
+                <mass value="${mass}"/>
                 <xacro:default_inertia />
             </inertial>
@@ -319,5 +320,5 @@
             <inertial>
                 <origin xyz="0 0 0" rpy="0 0 0"/>
-                <mass value="0.1"/>
+                <mass value="${mass}"/>
                 <xacro:default_inertia />
             </inertial>
@@ -349,5 +350,5 @@
             <inertial>
                 <origin xyz="0 0 0" rpy="0 0 0"/>
-                <mass value="0.1"/>
+                <mass value="${mass}"/>
                 <xacro:default_inertia />
             </inertial>
@@ -382,5 +383,5 @@
             <inertial>
                 <origin xyz="0 0 0" rpy="0 0 0"/>
-                <mass value="0.1"/>
+                <mass value="${mass}"/>
                 <xacro:default_inertia />
             </inertial>

Commit message: add xacro transmission param

File: hdt_description/urdf/hdt_angler_a_arm.xacro (robot description, xacro)
@@ -7,6 +7,6 @@
     <!-- camera sensor -->
     <xacro:include filename="$(find hdt_description)/urdf/hdt_angler_a_sensor.xacro" />
-    <xacro:macro name="hdt_serial_arm" params="namespace">
-        <xacro:hdt_transmission_macro namespace="${namespace}"/>
+    <xacro:macro name="hdt_serial_arm" params="namespace hardware_interface ">
+        <xacro:hdt_transmission_macro namespace="${namespace}" hardware_interface="${hardware_interface}" />
         <xacro:hdt_gazebo_macro namespace="${namespace}"/>
         <xacro:hdt_sensor_macro namespace="${namespace}"/>

Commit message: update mass value

File: hdt_description/urdf/hdt_angler_a_arm.xacro (robot description, xacro)
@@ -13,5 +13,5 @@
         <!-- constants -->
         <xacro:property name="M_PI" value="3.1415926535897931"/>
-        <xacro:property name="mass" value="0.107" />
+        <xacro:property name="mass" value="0.095" />
         <xacro:property name="drive_length" value="0.047"/>
         <xacro:property name="a35_length" value="0.03855"/>
@@ -55,11 +55,11 @@
                 <origin xyz="0 0 0" rpy="0 0 0"/>
                 <geometry>
-                    <mesh filename="package://hdt_angler_description/meshes/H026994 - A35 M-2 PEDESTAL ASSY - SHAREABLE.STL"/>
-                </geometry>
-            </collision>
-            <visual>
-                <origin xyz="0 0 0" rpy="0 0 0"/>
-                <geometry>
-                    <mesh filename="package://hdt_angler_description/meshes/H026994 - A35 M-2 PEDESTAL ASSY - SHAREABLE.STL"/>
+                    <mesh filename="package://hdt_description/meshes/H026994 - A35 M-2 PEDESTAL ASSY - SHAREABLE.STL"/>
+                </geometry>
+            </collision>
+            <visual>
+                <origin xyz="0 0 0" rpy="0 0 0"/>
+                <geometry>
+                    <mesh filename="package://hdt_description/meshes/H026994 - A35 M-2 PEDESTAL ASSY - SHAREABLE.STL"/>
                 </geometry>
                 <material name="black1"/>
@@ -84,11 +84,11 @@
                 <origin xyz="0 0 0" rpy="0 0 0"/>
                 <geometry>
-                    <mesh filename="package://hdt_angler_description/meshes/H024840 - A35 M-2 DRIVE MODULE, SHAREABLE.STL"/>
-                </geometry>
-            </collision>
-            <visual>
-                <origin xyz="0 0 0" rpy="0 0 0"/>
-                <geometry>
-                    <mesh filename="package://hdt_angler_description/meshes/H024840 - A35 M-2 DRIVE MODULE, SHAREABLE.STL"/>
+                    <mesh filename="package://hdt_description/meshes/H024840 - A35 M-2 DRIVE MODULE, SHAREABLE.STL"/>
+                </geometry>
+            </collision>
+            <visual>
+                <origin xyz="0 0 0" rpy="0 0 0"/>
+                <geometry>
+                    <mesh filename="package://hdt_description/meshes/H024840 - A35 M-2 DRIVE MODULE, SHAREABLE.STL"/>
                 </geometry>
                 <material name="black1"/>
@@ -113,11 +113,11 @@
                 <origin xyz="0 0 0" rpy="${M_PI} 0 0"/>
                 <geometry>
-                    <mesh filename="package://hdt_angler_description/meshes/H024840 - A35 M-2 DRIVE MODULE, SHAREABLE.STL"/>
-                </geometry>
-            </collision>
-            <visual>
-                <origin xyz="0 0 0" rpy="${M_PI} 0 0"/>
-                <geometry>
-                    <mesh filename="package://hdt_angler_description/meshes/H024840 - A35 M-2 DRIVE MODULE, SHAREABLE.STL"/>
+                    <mesh filename="package://hdt_description/meshes/H024840 - A35 M-2 DRIVE MODULE, SHAREABLE.STL"/>
+                </geometry>
+            </collision>
+            <visual>
+                <origin xyz="0 0 0" rpy="${M_PI} 0 0"/>
+                <geometry>
+                    <mesh filename="package://hdt_description/meshes/H024840 - A35 M-2 DRIVE MODULE, SHAREABLE.STL"/>
                 </geometry>
                 <material name="black1"/>
@@ -139,11 +139,11 @@
                 <origin xyz="0 0 0" rpy="0 0 0"/>
                 <geometry>
-                    <mesh filename="package://hdt_angler_description/meshes/H024847 - A35 M-2 PROXIMAL TUBE ASSY - SHAREABLE.STL"/>
-                </geometry>
-            </collision>
-            <visual>
-                <origin xyz="0 0 0" rpy="0 0 0"/>
-                <geometry>
-                    <mesh filename="package://hdt_angler_description/meshes/H024847 - A35 M-2 PROXIMAL TUBE ASSY - SHAREABLE.STL"/>
+                    <mesh filename="package://hdt_description/meshes/H024847 - A35 M-2 PROXIMAL TUBE ASSY - SHAREABLE.STL"/>
+                </geometry>
+            </collision>
+            <visual>
+                <origin xyz="0 0 0" rpy="0 0 0"/>
+                <geometry>
+                    <mesh filename="package://hdt_description/meshes/H024847 - A35 M-2 PROXIMAL TUBE ASSY - SHAREABLE.STL"/>
                 </geometry>
                 <material name="black1"/>
@@ -165,5 +165,5 @@
                 <origin xyz="0 0 0" rpy="0 ${M_PI} 0"/>
                 <geometry>
-                    <mesh filename="package://hdt_angler_description/meshes/H024840 - A35 M-2 DRIVE MODULE, SHAREABLE.STL"/>
+                    <mesh filename="package://hdt_description/meshes/H024840 - A35 M-2 DRIVE MODULE, SHAREABLE.STL"/>
                 </geometry>
             </collision>
@@ -171,5 +171,5 @@
                 <origin xyz="0 0 0" rpy="0 ${M_PI} 0"/>
                 <geometry>
-                    <mesh filename="package://hdt_angler_description/meshes/H024840 - A35 M-2 DRIVE MODULE, SHAREABLE.STL"/>
+                    <mesh filename="package://hdt_description/meshes/H024840 - A35 M-2 DRIVE MODULE, SHAREABLE.STL"/>
                 </geometry>
                 <material name="black1"/>
@@ -195,11 +195,11 @@
                 <origin xyz="0 0 0" rpy="0 ${M_PI/2} -${M_PI/2}"/>
                 <geometry>
-                    <mesh filename="package://hdt_angler_description/meshes/H024840 - A35 M-2 DRIVE MODULE, SHAREABLE.STL"/>
-                </geometry>
-            </collision>
-            <visual>
-                <origin xyz="0 0 0" rpy="0 ${M_PI/2} -${M_PI/2}"/>
-                <geometry>
-                    <mesh filename="package://hdt_angler_description/meshes/H024840 - A35 M-2 DRIVE MODULE, SHAREABLE.STL"/>
+                    <mesh filename="package://hdt_description/meshes/H024840 - A35 M-2 DRIVE MODULE, SHAREABLE.STL"/>
+                </geometry>
+            </collision>
+            <visual>
+                <origin xyz="0 0 0" rpy="0 ${M_PI/2} -${M_PI/2}"/>
+                <geometry>
+                    <mesh filename="package://hdt_description/meshes/H024840 - A35 M-2 DRIVE MODULE, SHAREABLE.STL"/>
                 </geometry>
                 <material name="black1"/>
@@ -224,11 +224,11 @@
                 <origin xyz="0 0 0" rpy="${M_PI} 0 0"/>
                 <geometry>
-                    <mesh filename="package://hdt_angler_description/meshes/H024848 - A35 M-2 DISTAL TUBE ASSY - SHAREABLE.STL"/>
-                </geometry>
-            </collision>
-            <visual>
-                <origin xyz="0 0 0" rpy="${M_PI} 0 0"/>
-                <geometry>
-                    <mesh filename="package://hdt_angler_description/meshes/H024848 - A35 M-2 DISTAL TUBE ASSY - SHAREABLE.STL"/>
+                    <mesh filename="package://hdt_description/meshes/H024848 - A35 M-2 DISTAL TUBE ASSY - SHAREABLE.STL"/>
+                </geometry>
+            </collision>
+            <visual>
+                <origin xyz="0 0 0" rpy="${M_PI} 0 0"/>
+                <geometry>
+                    <mesh filename="package://hdt_description/meshes/H024848 - A35 M-2 DISTAL TUBE ASSY - SHAREABLE.STL"/>
                 </geometry>
                 <material name="black1"/>
@@ -250,5 +250,5 @@
                 <origin xyz="0 0 0" rpy="0 0 ${M_PI}"/>
                 <geometry>
-                    <mesh filename="package://hdt_angler_description/meshes/H024840 - A35 M-2 DRIVE MODULE, SHAREABLE.STL"/>
+                    <mesh filename="package://hdt_description/meshes/H024840 - A35 M-2 DRIVE MODULE, SHAREABLE.STL"/>
                 </geometry>
             </collision>
@@ -256,5 +256,5 @@
                 <origin xyz="0 0 0" rpy="0 0 ${M_PI}"/>
                 <geometry>
-                    <mesh filename="package://hdt_angler_description/meshes/H024840 - A35 M-2 DRIVE MODULE, SHAREABLE.STL"/>
+                    <mesh filename="package://hdt_description/meshes/H024840 - A35 M-2 DRIVE MODULE, SHAREABLE.STL"/>
                 </geometry>
                 <material name="black1"/>
@@ -279,5 +279,5 @@
                 <origin xyz="0 0 0" rpy="0 ${M_PI/2} ${M_PI}"/>
                 <geometry>
-                    <mesh filename="package://hdt_angler_description/meshes/H024840 - A35 M-2 DRIVE MODULE, SHAREABLE.STL"/>
+                    <mesh filename="package://hdt_description/meshes/H024840 - A35 M-2 DRIVE MODULE, SHAREABLE.STL"/>
                 </geometry>
             </collision>
@@ -285,5 +285,5 @@
                 <origin xyz="0 0 0" rpy="0 ${M_PI/2} ${M_PI}"/>
                 <geometry>
-                    <mesh filename="package://hdt_angler_description/meshes/H024840 - A35 M-2 DRIVE MODULE, SHAREABLE.STL"/>
+                    <mesh filename="package://hdt_description/meshes/H024840 - A35 M-2 DRIVE MODULE, SHAREABLE.STL"/>
                 </geometry>
                 <material name="black1"/>
@@ -308,11 +308,11 @@
                 <origin xyz="0 0 0" rpy="0 ${M_PI/2} -${M_PI/2}"/>
                 <geometry>
-                    <mesh filename="package://hdt_angler_description/meshes/H024842 - A35 M-2 PINCER ASSY - SHAREABLE, UNDERWATER.STL"/>
-                </geometry>
-            </collision>
-            <visual>
-                <origin xyz="0 0 0" rpy="0 ${M_PI/2} -${M_PI/2}"/>
-                <geometry>
-                    <mesh filename="package://hdt_angler_description/meshes/H024842 - A35 M-2 PINCER ASSY - SHAREABLE, UNDERWATER.STL"/>
+                    <mesh filename="package://hdt_description/meshes/H024842 - A35 M-2 PINCER ASSY - SHAREABLE, UNDERWATER.STL"/>
+                </geometry>
+            </collision>
+            <visual>
+                <origin xyz="0 0 0" rpy="0 ${M_PI/2} -${M_PI/2}"/>
+                <geometry>
+                    <mesh filename="package://hdt_description/meshes/H024842 - A35 M-2 PINCER ASSY - SHAREABLE, UNDERWATER.STL"/>
                 </geometry>
                 <material name="black1"/>
@@ -338,11 +338,11 @@
                 <origin xyz="0 0 0" rpy="${M_PI} 0 0"/>
                 <geometry>
-                    <mesh filename="package://hdt_angler_description/meshes/H022927 - A35 PINCER FINGER, LONG, OVERMOLD ASSY - SHAREABLE.STL"/>
-                </geometry>
-            </collision>
-            <visual>
-                <origin xyz="0 0 0" rpy="${M_PI} 0 0"/>
-                <geometry>
-                    <mesh filename="package://hdt_angler_description/meshes/H022927 - A35 PINCER FINGER, LONG, OVERMOLD ASSY - SHAREABLE.STL"/>
+                    <mesh filename="package://hdt_description/meshes/H022927 - A35 PINCER FINGER, LONG, OVERMOLD ASSY - SHAREABLE.STL"/>
+                </geometry>
+            </collision>
+            <visual>
+                <origin xyz="0 0 0" rpy="${M_PI} 0 0"/>
+                <geometry>
+                    <mesh filename="package://hdt_description/meshes/H022927 - A35 PINCER FINGER, LONG, OVERMOLD ASSY - SHAREABLE.STL"/>
                 </geometry>
                 <material name="black1"/>
@@ -371,11 +371,11 @@
                 <origin xyz="0 0 0" rpy="${M_PI} 0 0"/>
                 <geometry>
-                <mesh filename="package://hdt_angler_description/meshes/H022927 - A35 PINCER FINGER, LONG, OVERMOLD ASSY - SHAREABLE.STL"/>
-                </geometry>
-            </collision>
-            <visual>
-                <origin xyz="0 0 0" rpy="${M_PI} 0 0"/>
-                <geometry>
-                    <mesh filename="package://hdt_angler_description/meshes/H022927 - A35 PINCER FINGER, LONG, OVERMOLD ASSY - SHAREABLE.STL"/>
+                <mesh filename="package://hdt_description/meshes/H022927 - A35 PINCER FINGER, LONG, OVERMOLD ASSY - SHAREABLE.STL"/>
+                </geometry>
+            </collision>
+            <visual>
+                <origin xyz="0 0 0" rpy="${M_PI} 0 0"/>
+                <geometry>
+                    <mesh filename="package://hdt_description/meshes/H022927 - A35 PINCER FINGER, LONG, OVERMOLD ASSY - SHAREABLE.STL"/>
                 </geometry>
                 <material name="black1"/>
